File: board/radar.kicad_pcb (KiCad board)
At the start: 2 copper layers, 83 parts, among them K1 CONN_3, K2 CONN_3, P1 CONN_2, P2 CONN_7, P3 CONN_8, Q1 2N3906, Q2 MOSFET_P, Q3 MOSFET_P, U1 ATMEGA8-P, U2 LM7805, U3 TLE2021, U4 LM78L03ACZ, U5 LM358, X1 16MHz

Commit message: Finish pcb layout
Parts:
- removed R26: 47k, R4
- moved R5 259.8 mm to (269.9, 158.1), turned to 270 degrees
- moved P1 254.3 mm to (275.0, 128.9), turned to 90 degrees
- moved F1 253.8 mm to (275.0, 150.5), turned to 270 degrees
- moved L1 251.1 mm to (269.9, 144.1)
- moved D1 243.3 mm to (275.0, 135.9), turned to 180 degrees
- moved D2 234.4 mm to (262.3, 134.0), turned to 180 degrees
- moved U2 225.8 mm to (262.3, 126.4)
- moved C8 224.1 mm to (259.7, 139.7)
- moved C10 223.5 mm to (259.7, 131.4)
- moved C12 200.7 mm to (199.4, 127.0)
- moved C17 200.3 mm to (212.7, 135.9)
- moved C11 199.6 mm to (208.3, 142.2)
- moved R10 199.6 mm to (196.2, 134.6)
- moved R12 199.6 mm to (198.8, 134.6)
- moved R14 199.6 mm to (198.1, 124.5)
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Connections:
- C9 pad 1: N-0000054 -> +5V
- R9 pad 2: N-0000054 -> +5V
- U1 pad 24: /radar_60db -> /radar_80db
- U1 pad 25: /radar_80db -> /radar_100db
- U1 pad 26: /radar_100db -> /radar_60db
- U1 pad 4: /DISPLAY_RST -> /DISPLAY_DC
- U1 pad 5: /DISPLAY_DC -> /DISPLAY_CS
- U1 pad 6: /DISPLAY_CS -> /DISPLAY_RST
- U1 pad 7: N-0000054 -> +5V
Routing:
- net GND: track 35.0 -> 467.0 mm, vias 0 -> 2
- net +5V: track 0.00 -> 267.3 mm, vias 0 -> 8
- net /RESET: track 0.00 -> 83.8 mm
- net /MOSI: track 0.00 -> 64.0 mm
- net /SCK: track 0.00 -> 58.1 mm
- net /DISPLAY_LED: track 0.00 -> 57.4 mm, vias 0 -> 1
- net /RADAR_EN: track 0.00 -> 56.9 mm, vias 0 -> 2
- net /radar_100db: track 0.00 -> 49.9 mm, vias 0 -> 2
- net /KEYBOARD: track 0.00 -> 47.3 mm, vias 0 -> 4
- net N-0000056: track 0.00 -> 46.0 mm, vias 0 -> 2
- net /radar_60db: track 0.00 -> 43.5 mm, vias 0 -> 2
- net /DISPLAY_CS: track 0.00 -> 40.2 mm
- net /DISPLAY_DC: track 0.00 -> 40.0 mm
- net /DISPLAY_RST: track 0.00 -> 39.1 mm
- net N-0000014: track 0.00 -> 34.2 mm
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- added copper zone on B.Cu, net GND
Other:
- board outline added: 108 x 57.1 mm
- net class Small added: clearance 0.254, trace_width 0.254, via_dia 0.889, via_drill 0.635
