File: board/data-logger.kicad_pcb (KiCad board)
At the start: 4 copper layers, 207 parts, among them P401 CONN_01X02, P402 CONN_01X02, P403 CONN_01X04, P501 CONN_02X03, P502 CONN_02X06, P503 MICROSD, P504 USB_B, P601 CONN_02X08, P602 CONN_02X08, P603 CONN_02X08, P604 CONN_02X08, Q401 IRLML6401, Q501 IRLML6401, U201 10M08DCF256, U202 AS4C8M16SA-7TCN, U203 AS4C8M16SA-7TCN, U302 SAM3U1EB-CU, U401 LM4120, U402 BQ24161RGE, U403 TPS62097, U404 TPS62097, U405 TPS76325, U406 TPS63001, U501 LSF0204, U502 LSF0204, U601 MCP6002, X501 CONN_DEBUG_MCNET, X502 IQXO/7X, Y501 32.768 kHz, Y502 12.000 MHz

Commit message: Some initial layout work
Parts:
- removed JP401: JUMPER, Pin_Headers:Pin_Header_Straight_1x02_Pitch2.54mm
- added BT401: CR3202, AMesser_Connectors:keystone_electronics_106, F.Cu at (28.7, 64.7)
- added C437: 4.7µF, Capacitors_SMD:C_0402, F.Cu at (80.9, 139.4)
- added C438: 4.7µF, Capacitors_SMD:C_0402, F.Cu at (91.0, 142.1)
- added C439: 4.7µF, Capacitors_SMD:C_0402, F.Cu at (54.5, 141.8)
- added C440: 4.7µF, Capacitors_SMD:C_0402, F.Cu at (46.5, 142.2)
- added C441: 4.7µF, Capacitors_SMD:C_0402, F.Cu at (90.2, 96.8)
- added C516: 100nF, Capacitors_SMD:C_0805, F.Cu at (6.70, 102.7)
- added Q402: Q_NMOS_GSD, TO_SOT_Packages_SMD:SOT-23, F.Cu at (57.5, 136.9)
- added REF**: MountingHole_3.5mm_Pad, Mounting_Holes:MountingHole_3.5mm_Pad, F.Cu at (106.5, 43.5)
- added REF**: MountingHole_3.5mm_Pad, Mounting_Holes:MountingHole_3.5mm_Pad, F.Cu at (46.5, 43.5)
- added REF**: MountingHole_3.5mm_Pad, Mounting_Holes:MountingHole_3.5mm_Pad, F.Cu at (46.5, 123.5)
- added REF**: MountingHole_3.5mm_Pad, Mounting_Holes:MountingHole_3.5mm_Pad, F.Cu at (106.5, 123.5)
- added U407: TPS63001, AMesser_Power_Management:Texas_Instruments_PVSON-N10, F.Cu at (34.7, 45.7)
- C402: value 22n -> 1µF; footprint Capacitors_SMD:C_0402 -> Capacitors_SMD:C_0603
- C404: value 1µF -> 4.7µF; footprint Capacitors_SMD:C_0603 -> Capacitors_SMD:C_0402
- C406: value 4.7µF -> 22n; footprint Capacitors_SMD:C_0402 -> Capacitors_SMD:C_0603
- C409: footprint Capacitors_SMD:C_0603 -> Capacitors_SMD:C_0402
- C410: value 4.7µF -> 1µF
- C411: value 4.7µF -> 1µF; footprint Capacitors_SMD:C_0402 -> Capacitors_SMD:C_0603
- C414, C510: value 100nF -> 4.7µF
- C415: value 10nF -> 4.7µF; footprint Capacitors_SMD:C_0402 -> Capacitors_SMD:C_0603
- C416: value 10µF -> 4.7µF
- C417, C418: value 10µF -> 4.7µF; footprint Capacitors_SMD:C_0603 -> Capacitors_SMD:C_0402
- C419: value 10µF -> 100nF
- C420, C427: value 10µF -> 10nF
- C422: value 1µF -> 10µF
- C423: value 10nF -> 10µF; footprint Capacitors_SMD:C_0402 -> Capacitors_SMD:C_0603
- C428, C429: value 10µF -> 1µF
- C431, C432, C433, C434, C435: value 4.7µF -> 10µF; footprint Capacitors_SMD:C_0402 -> Capacitors_SMD:C_0603
- C509: value 4.7µF -> 10nF; footprint Capacitors_SMD:C_0402 -> Capacitors_SMD:C_0603
- C511, C603: footprint Capacitors_SMD:C_0402 -> Capacitors_SMD:C_0603
- C512: value 10pF -> 100nF; footprint Capacitors_SMD:C_0402 -> Capacitors_SMD:C_0603
- C513: value 100nF -> 10pF
- C514: value 4.7µF -> 100nF; footprint Capacitors_SMD:C_0402 -> Capacitors_SMD:C_0805
- C515: value 100nF -> 4.7µF; footprint Capacitors_SMD:C_0603 -> Capacitors_SMD:C_0402
- C601: value 4.7 µF -> 4.7µF
- C607: value 100 nF -> 100nF; footprint Capacitors_SMD:C_0402 -> Capacitors_SMD:C_0603
- C608: value 4.7µF -> 100nF; footprint Capacitors_SMD:C_0402 -> Capacitors_SMD:C_0603
- D401: value D_Schottky -> BAT54C; footprint Diodes_SMD:D_SMA_Standard -> TO_SOT_Packages_SMD:SOT-23
- D402: value ZENER -> D_Schottky
- D403: value Led_Small -> ZENER; footprint LEDs:LED_0805 -> Diodes_SMD:D_SMA_Standard
- D404: value BAT54C -> Led_Small; footprint TO_SOT_Packages_SMD:SOT-23 -> LEDs:LED_0805
- P401: footprint Connectors_Phoenix:PhoenixContact_MSTBVA-G_02x5.00mm_Vertical -> Connectors_JST:JST_EH_B02B-EH-A_02x2.50mm_Straight
- P402: value CONN_01X02 -> CONN_01X04; footprint Pin_Headers:Pin_Header_Straight_1x02_Pitch2.54mm -> Connectors_JST:JST_EH_B04B-EH-A_04x2.50mm_Straight
- P403: footprint Pin_Headers:Pin_Header_Straight_1x04_Pitch2.54mm -> Connectors_JST:JST_EH_B04B-EH-A_04x2.50mm_Straight
- P601, P602, P603, P604: footprint Pin_Headers:Pin_Header_Straight_2x08_Pitch2.54mm -> Pin_Headers:Pin_Header_Angled_2x08_Pitch2.54mm
- R201, R202, R203, R204, R205, R206, R207, R208, R301, R302, R303, R402, R501, R502, R505, R506, R507, R514, R602, R603, R604, R605, R606, R607, R608, R609, R610, R611, R612, R613: footprint Resistors_SMD:R_Array_Concave_4x0402 -> Resistors_SMD:R_Array_Convex_4x0603
- R404: value 100k -> 1
- R405: value 1 -> 100k; footprint Resistors_SMD:R_0603 -> Resistors_SMD:R_Array_Convex_4x0603
- R406: value 100 -> 1.0k
- R407: value 1.0k -> 100
- U302: value SAM3U1EB-CU -> SAM3U1EB-AU; footprint board_footprints:LFBGA_144 -> Housings_QFP:LQFP-144_20x20mm_Pitch0.5mm
- U401: value LM4120 -> AP2138N-2.5TRG1; footprint TO_SOT_Packages_SMD:SOT-23-5 -> TO_SOT_Packages_SMD:SOT-23
- U402: value BQ24161RGE -> LM4120; footprint board_footprints:VQFN-24_EP -> TO_SOT_Packages_SMD:SOT-23-5
- U403: value TPS62097 -> BQ24161RGE; footprint AMesser_Power_Management:Texas_Instruments_VQFN-HR-11 -> board_footprints:VQFN-24_EP
- U405: value TPS76325 -> TPS62097; footprint TO_SOT_Packages_SMD:SOT-23-5 -> AMesser_Power_Management:Texas_Instruments_VQFN-HR-11
- U406: value TPS63001 -> AP2138N-2.5TRG1; footprint AMesser_Power_Management:Texas_Instruments_PVSON-N10 -> TO_SOT_Packages_SMD:SOT-23
- X501: footprint Pin_Headers:Pin_Header_Angled_2x05_Pitch2.54mm -> Pin_Headers:Pin_Header_Straight_2x05_Pitch2.54mm
- Y502: value 12.000 MHz -> 12.000MHz
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Connections:
- C401 pad 1: Net-(C401-Pad1) -> /Power Supply/VCC_SYS
- C402 pad 1: /Power Supply/VREF_2V5 -> Net-(C402-Pad1)
- C403 pad 1: +1V8 -> VCCIO_MCU
- C404 pad 1: Net-(C404-Pad1) -> +1V8
- C405 pad 1: VCC_USB -> Net-(C405-Pad1)
- C406 pad 1: VCCIO_MCU -> /Power Supply/VREF_2V5
- C407 pad 1: +1V8 -> VCCIO_MCU
- C408 pad 1: Net-(C408-Pad1) -> VCCBU_MCU
- C409 pad 1: Net-(C409-Pad1) -> +1V8
- C411 pad 1: /Power Supply/VCCBU_MCU -> VCC_USB
- C415 pad 2: Net-(C415-Pad2) -> GND
- C417 pad 1: /Power Supply/VCC_SYS -> VCCIO_MCU
- C418 pad 1: /Power Supply/VCC_SYS -> +1V8
- C420 pad 1: Net-(C419-Pad1) -> Net-(C420-Pad1)
- C420 pad 2: GND -> Net-(C420-Pad2)
- C421 pad 1: Net-(C419-Pad1) -> Net-(C421-Pad1)
- C422 pad 1: Net-(C419-Pad1) -> /Power Supply/VCC_SYS
- C423 pad 1: Net-(C423-Pad1) -> /Power Supply/VCC_SYS
- C424 pad 1: +2V5 -> Net-(C424-Pad1)
- C425 pad 1: VCCIO_MCU -> Net-(C424-Pad1)
- C426 pad 1: +1V8 -> Net-(C424-Pad1)
- C427 pad 1: +1V2 -> Net-(C427-Pad1)
- C429 pad 1: +1V8 -> +2V5
- C430 pad 1: +1V2 -> VCCIO_MCU
- C431 pad 1: +1V2 -> +1V8
- C433 pad 1: +1V2 -> VCCIO_MCU
- C434 pad 1: +1V2 -> +1V8
- C435 pad 1: Net-(C435-Pad1) -> +1V2
- C436 pad 1: Net-(C436-Pad1) -> +1V2
- C511 pad 1: VCCIO_MCU -> Net-(C511-Pad1)
- C512 pad 1: Net-(C512-Pad1) -> VCCIO_MCU
- D401 pad 1: Net-(C404-Pad1) -> Net-(BT401-Pad1)
- D401 pad 2: Net-(D401-Pad2) -> Net-(C402-Pad1)
- D402 pad 1: Net-(C404-Pad1) -> Net-(C410-Pad1)
- D402 pad 2: GND -> Net-(D402-Pad2)
- D403 pad 1: Net-(D403-Pad1) -> Net-(C410-Pad1)
- D403 pad 2: Net-(C401-Pad1) -> GND
- D404 pad 1: VCCIO_MCU -> Net-(D404-Pad1)
- D404 pad 2: Net-(D404-Pad2) -> Net-(C405-Pad1)
- D405 pad 2: Net-(C419-Pad1) -> VCCIO_MCU
- JP502 pad 1: GND -> Net-(C509-Pad1)
- JP502 pad 2: Net-(JP502-Pad2) -> GND
- L401 pad 1: VCCIO_MCU -> Net-(C419-Pad1)
- L401 pad 2: Net-(C414-Pad1) -> VCCIO_MCU
- L402 pad 1: Net-(C415-Pad1) -> Net-(C420-Pad1)
- L406 pad 1: Net-(C435-Pad1) -> Net-(C440-Pad1)
- L407 pad 1: Net-(C436-Pad1) -> Net-(C441-Pad1)
- L501 pad 2: Net-(C510-Pad1) -> Net-(C511-Pad1)
- L502 pad 2: Net-(C514-Pad1) -> Net-(C515-Pad1)
- P402 pad 1: Net-(D404-Pad2) -> /Power Supply/VCC_SYS
- P402 pad 2: GND -> Net-(C424-Pad1)
- P403 pad 1: Net-(C416-Pad1) -> Net-(C421-Pad1)
- P403 pad 4: Net-(C401-Pad1) -> Net-(C405-Pad1)
- P503 pad 4: Net-(C514-Pad1) -> Net-(C515-Pad1)
- P503 pad S: Net-(C513-Pad1) -> Net-(C514-Pad1)
- P504 pad 5: Net-(C515-Pad1) -> Net-(C516-Pad1)
- Q401 pad 3: Net-(C416-Pad1) -> Net-(C421-Pad1)
- R201 pad 1: Net-(R201-Pad1) -> /SDRAM/SDRAM_D0
- R201 pad 2: Net-(R201-Pad2) -> /SDRAM/SDRAM_D1
- R201 pad 3: Net-(R201-Pad3) -> /SDRAM/SDRAM_D2
- R201 pad 4: Net-(R201-Pad4) -> /SDRAM/SDRAM_D3
- R201 pad 5: /SDRAM/SDRAM_D3 -> Net-(R201-Pad5)
- R201 pad 6: /SDRAM/SDRAM_D2 -> Net-(R201-Pad6)
- R201 pad 7: /SDRAM/SDRAM_D1 -> Net-(R201-Pad7)
- R201 pad 8: /SDRAM/SDRAM_D0 -> Net-(R201-Pad8)
- R202 pad 1: Net-(R202-Pad1) -> /SDRAM/SDRAM_D4
- R202 pad 2: Net-(R202-Pad2) -> /SDRAM/SDRAM_D5
- R202 pad 3: Net-(R202-Pad3) -> /SDRAM/SDRAM_D6
- R202 pad 4: Net-(R202-Pad4) -> /SDRAM/SDRAM_D7
- R202 pad 5: /SDRAM/SDRAM_D7 -> Net-(R202-Pad5)
- R202 pad 6: /SDRAM/SDRAM_D6 -> Net-(R202-Pad6)
- R202 pad 7: /SDRAM/SDRAM_D5 -> Net-(R202-Pad7)
- R202 pad 8: /SDRAM/SDRAM_D4 -> Net-(R202-Pad8)
- R203 pad 5: /SDRAM/SDRAM_D11 -> /SDRAM/SDRAM_D8
- R203 pad 6: /SDRAM/SDRAM_D10 -> /SDRAM/SDRAM_D9
- R203 pad 7: /SDRAM/SDRAM_D9 -> /SDRAM/SDRAM_D10
- R203 pad 8: /SDRAM/SDRAM_D8 -> /SDRAM/SDRAM_D11
- R204 pad 5: /SDRAM/SDRAM_D15 -> /SDRAM/SDRAM_D12
- R204 pad 6: /SDRAM/SDRAM_D14 -> /SDRAM/SDRAM_D13
- R204 pad 7: /SDRAM/SDRAM_D13 -> /SDRAM/SDRAM_D14
- R204 pad 8: /SDRAM/SDRAM_D12 -> /SDRAM/SDRAM_D15
- R205 pad 1: Net-(R205-Pad1) -> /SDRAM/SDRAM_D16
- R205 pad 2: Net-(R205-Pad2) -> /SDRAM/SDRAM_D17
- R205 pad 3: Net-(R205-Pad3) -> /SDRAM/SDRAM_D18
- R205 pad 4: Net-(R205-Pad4) -> /SDRAM/SDRAM_D19
- R205 pad 5: /SDRAM/SDRAM_D19 -> Net-(R205-Pad5)
- R205 pad 6: /SDRAM/SDRAM_D18 -> Net-(R205-Pad6)
- R205 pad 7: /SDRAM/SDRAM_D17 -> Net-(R205-Pad7)
- R205 pad 8: /SDRAM/SDRAM_D16 -> Net-(R205-Pad8)
- R206 pad 1: Net-(R206-Pad1) -> /SDRAM/SDRAM_D20
- R206 pad 2: Net-(R206-Pad2) -> /SDRAM/SDRAM_D21
- R206 pad 3: Net-(R206-Pad3) -> /SDRAM/SDRAM_D22
- R206 pad 4: Net-(R206-Pad4) -> /SDRAM/SDRAM_D23
- R206 pad 5: /SDRAM/SDRAM_D23 -> Net-(R206-Pad5)
- R206 pad 6: /SDRAM/SDRAM_D22 -> Net-(R206-Pad6)
- R206 pad 7: /SDRAM/SDRAM_D21 -> Net-(R206-Pad7)
- R206 pad 8: /SDRAM/SDRAM_D20 -> Net-(R206-Pad8)
- R207 pad 5: /SDRAM/SDRAM_D27 -> /SDRAM/SDRAM_D24
- R207 pad 6: /SDRAM/SDRAM_D26 -> /SDRAM/SDRAM_D25
- R207 pad 7: /SDRAM/SDRAM_D25 -> /SDRAM/SDRAM_D26
- R207 pad 8: /SDRAM/SDRAM_D24 -> /SDRAM/SDRAM_D27
- R208 pad 5: /SDRAM/SDRAM_D31 -> /SDRAM/SDRAM_D28
- R208 pad 6: /SDRAM/SDRAM_D30 -> /SDRAM/SDRAM_D29
- R208 pad 7: /SDRAM/SDRAM_D29 -> /SDRAM/SDRAM_D30
- R208 pad 8: /SDRAM/SDRAM_D28 -> /SDRAM/SDRAM_D31
- R303 pad 1: Net-(D301-Pad2) -> Net-(D304-Pad2)
- R303 pad 2: Net-(D302-Pad2) -> Net-(D303-Pad2)
- R303 pad 3: Net-(D303-Pad2) -> Net-(D302-Pad2)
- R303 pad 4: Net-(D304-Pad2) -> Net-(D301-Pad2)
- R401 pad 1: Net-(D401-Pad2) -> Net-(D402-Pad2)
- R403 pad 1: Net-(D403-Pad1) -> Net-(D404-Pad1)
- R404 pad 1: /Power Supply/VCCBU_MCU -> Net-(C414-Pad1)
- R404 pad 2: Net-(R404-Pad2) -> Net-(C419-Pad1)
- R405 pad 1: Net-(C408-Pad1) -> VCCBU_MCU
- R405 pad 2: Net-(C414-Pad1) -> Net-(Q402-Pad1)
- R406 pad 1: Net-(C419-Pad1) -> GND
- R406 pad 2: Net-(C423-Pad1) -> Net-(D405-Pad1)
- R407 pad 1: GND -> Net-(C424-Pad1)
- R407 pad 2: Net-(D405-Pad1) -> Net-(C427-Pad1)
- R502 pad 1: Net-(D501-Pad2) -> Net-(D504-Pad2)
- R502 pad 2: Net-(D502-Pad2) -> Net-(D503-Pad2)
- R502 pad 3: Net-(D503-Pad2) -> Net-(D502-Pad2)
- R502 pad 4: Net-(D504-Pad2) -> Net-(D501-Pad2)
- R505 pad 3: Net-(JP501-Pad3) -> VCCBU_MCU
- R505 pad 4: GND -> Net-(JP501-Pad3)
- R505 pad 5: Net-(R505-Pad5) -> VCCIO_MCU
- R505 pad 6: VCCIO_MCU -> Net-(C509-Pad1)
- R506 pad 1: Net-(JP502-Pad2) -> GND
- R506 pad 2: GND -> Net-(R506-Pad2)
- R506 pad 3: Net-(R506-Pad3) -> GND
- R506 pad 6: VCCIO_MCU -> Net-(R506-Pad6)
- R506 pad 7: Net-(R506-Pad7) -> VCCIO_MCU
- R506 pad 8: VCCIO_MCU -> Net-(R506-Pad8)
- R507 pad 3: (no net) -> Net-(C601-Pad1)
- R507 pad 4: (no net) -> GND
- R507 pad 5: (no net) -> Net-(C603-Pad1)
- R507 pad 6: (no net) -> Net-(C603-Pad1)
- R507 pad 7: Net-(C514-Pad1) -> Net-(C515-Pad1)
- R508 pad 1: Net-(C510-Pad1) -> Net-(C511-Pad1)
- R508 pad 2: Net-(C509-Pad1) -> Net-(C510-Pad1)
- R509 pad 1: Net-(C512-Pad1) -> Net-(C513-Pad1)
- R514 pad 5: Net-(C514-Pad1) -> Net-(C515-Pad1)
- R514 pad 6: Net-(C514-Pad1) -> Net-(C515-Pad1)
- R514 pad 7: Net-(C514-Pad1) -> Net-(C515-Pad1)
- R514 pad 8: Net-(C514-Pad1) -> Net-(C515-Pad1)
- R515 pad 2: Net-(C513-Pad1) -> Net-(C514-Pad1)
- R518 pad 2: Net-(C515-Pad1) -> Net-(C516-Pad1)
- R610 pad 3: Net-(C601-Pad1) -> (no net)
- R610 pad 4: GND -> (no net)
- R610 pad 5: Net-(C603-Pad1) -> (no net)
- R610 pad 6: Net-(C603-Pad1) -> (no net)
- U201 pad A13: /SDRAM/~SDRAM_CAS~ -> /SDRAM/SDRAM_D31
- U201 pad D13: Net-(C435-Pad1) -> Net-(C440-Pad1)
- U201 pad D5: Net-(C436-Pad1) -> Net-(C441-Pad1)
- U201 pad E12: Net-(C436-Pad1) -> Net-(C441-Pad1)
- U201 pad E16: /SDRAM/SDRAM_D31 -> /SDRAM/~SDRAM_CAS~
- U201 pad E4: Net-(C436-Pad1) -> Net-(C441-Pad1)
- U201 pad E5: Net-(C436-Pad1) -> Net-(C441-Pad1)
- U201 pad K5: MCU_NPCS2 -> ~MCU_NPCS2~
- U201 pad K8: Net-(U201-PadK8) -> +1V2
- U201 pad L2: MCU_NPCS1 -> ~MCU_NPCS1~
- U201 pad L5: Net-(C436-Pad1) -> Net-(C441-Pad1)
- U201 pad M12: Net-(C436-Pad1) -> Net-(C441-Pad1)
- U201 pad M2: MCU_NPCS0 -> ~MCU_NPCS0~
- U201 pad M5: Net-(C435-Pad1) -> Net-(C440-Pad1)
- U202 pad 10: Net-(R202-Pad2) -> Net-(R202-Pad7)
- U202 pad 11: Net-(R202-Pad3) -> Net-(R202-Pad6)
- U202 pad 13: Net-(R202-Pad4) -> Net-(R202-Pad5)
- U202 pad 2: Net-(R201-Pad1) -> Net-(R201-Pad8)
- U202 pad 4: Net-(R201-Pad2) -> Net-(R201-Pad7)
- U202 pad 42: Net-(R203-Pad1) -> Net-(R203-Pad4)
- U202 pad 44: Net-(R203-Pad2) -> Net-(R203-Pad3)
- U202 pad 45: Net-(R203-Pad3) -> Net-(R203-Pad2)
- U202 pad 47: Net-(R203-Pad4) -> Net-(R203-Pad1)
- U202 pad 48: Net-(R204-Pad1) -> Net-(R204-Pad4)
- U202 pad 5: Net-(R201-Pad3) -> Net-(R201-Pad6)
- U202 pad 50: Net-(R204-Pad2) -> Net-(R204-Pad3)
- U202 pad 51: Net-(R204-Pad3) -> Net-(R204-Pad2)
- U202 pad 53: Net-(R204-Pad4) -> Net-(R204-Pad1)
- U202 pad 7: Net-(R201-Pad4) -> Net-(R201-Pad5)
- U202 pad 8: Net-(R202-Pad1) -> Net-(R202-Pad8)
- U203 pad 10: Net-(R206-Pad2) -> Net-(R206-Pad7)
- U203 pad 11: Net-(R206-Pad3) -> Net-(R206-Pad6)
- U203 pad 13: Net-(R206-Pad4) -> Net-(R206-Pad5)
- U203 pad 2: Net-(R205-Pad1) -> Net-(R205-Pad8)
- U203 pad 4: Net-(R205-Pad2) -> Net-(R205-Pad7)
- U203 pad 42: Net-(R207-Pad1) -> Net-(R207-Pad4)
- U203 pad 44: Net-(R207-Pad2) -> Net-(R207-Pad3)
- U203 pad 45: Net-(R207-Pad3) -> Net-(R207-Pad2)
- U203 pad 47: Net-(R207-Pad4) -> Net-(R207-Pad1)
- U203 pad 48: Net-(R208-Pad1) -> Net-(R208-Pad4)
- U203 pad 5: Net-(R205-Pad3) -> Net-(R205-Pad6)
- U203 pad 50: Net-(R208-Pad2) -> Net-(R208-Pad3)
- U203 pad 51: Net-(R208-Pad3) -> Net-(R208-Pad2)
- U203 pad 53: Net-(R208-Pad4) -> Net-(R208-Pad1)
- U203 pad 7: Net-(R205-Pad4) -> Net-(R205-Pad5)
- U203 pad 8: Net-(R206-Pad1) -> Net-(R206-Pad8)
- U401 pad 1: Net-(U401-Pad1) -> GND
- U401 pad 2: GND -> Net-(C402-Pad1)
- U401 pad 3: Net-(C414-Pad1) -> /Power Supply/VCC_SYS
- U402 pad 1: (no net) -> Net-(U402-Pad1)
- U402 pad 2: Net-(C401-Pad1) -> GND
- U402 pad 3: MCU_TWCK0 -> Net-(C419-Pad1)
- U402 pad 4: MCU_TWD0 -> Net-(C419-Pad1)
- U402 pad 5: GND -> /Power Supply/VREF_2V5
- U403 pad 1: GND -> (no net)
- U403 pad 10: GND -> Net-(Q401-Pad1)
- U403 pad 11: GND -> Net-(C421-Pad1)
- U403 pad 2: Net-(L404-Pad1) -> Net-(C405-Pad1)
- U403 pad 3: +1V8 -> MCU_TWCK0
- U403 pad 4: Net-(R412-Pad1) -> MCU_TWD0
- U403 pad 5: Net-(U403-Pad5) -> GND
- U403 pad 6: Net-(C419-Pad1) -> Net-(C405-Pad1)
- U403 pad 7: Net-(C419-Pad1) -> MCU_PWRINT
- U403 pad 8: Net-(C419-Pad1) -> Net-(R403-Pad2)
- U403 pad 9: Net-(R408-Pad2) -> Net-(P403-Pad3)
- U404 pad 2: Net-(L405-Pad1) -> Net-(L404-Pad1)
- U404 pad 3: +1V2 -> +1V8
- U404 pad 4: Net-(R413-Pad1) -> Net-(R412-Pad1)
- U404 pad 6: Net-(C419-Pad1) -> Net-(C424-Pad1)
- U404 pad 7: Net-(C419-Pad1) -> Net-(C424-Pad1)
- U404 pad 8: Net-(C419-Pad1) -> Net-(C424-Pad1)
- U404 pad 9: Net-(R410-Pad2) -> Net-(R408-Pad2)
- U405 pad 1: Net-(C419-Pad1) -> GND
- U405 pad 2: GND -> Net-(L405-Pad1)
- U405 pad 3: Net-(C419-Pad1) -> +1V2
- U405 pad 4: +2V5 -> Net-(R413-Pad1)
- U405 pad 5: +2V5 -> Net-(U405-Pad5)
- U406 pad 1: VCCIO_MCU -> GND
- U406 pad 2: Net-(L403-Pad2) -> +2V5
- U406 pad 3: GND -> VCCIO_MCU
- U501 pad 12: Net-(R506-Pad7) -> Net-(R506-Pad6)
- U501 pad 13: Net-(R506-Pad3) -> Net-(R506-Pad2)
- W401 pad 1: Net-(C401-Pad1) -> Net-(C405-Pad1)
- X501 pad 3: Net-(R506-Pad7) -> Net-(R506-Pad6)
- X501 pad 5: Net-(R506-Pad3) -> Net-(R506-Pad2)
- X501 pad 6: Net-(U302-PadD9) -> Net-(U302-Pad1)
- Y502 pad 2: Net-(C508-Pad1) -> GND
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Routing:
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Other:
- board outline added: 105 x 100 mm
- net class Default: clearance 0.2 -> 0.125; trace_width 0.25 -> 0.125; via_drill 0.4 -> 0.3
- net class Standard Signal added: clearance 0.2, trace_width 0.3, via_dia 0.6, via_drill 0.3
- rule pad_to_mask_clearance: 0.2 -> 0.1
- rule trace_clearance: 0.2 -> 0.125
- rule trace_min: 0.2 -> 0.125
- rule via_min_drill: 0.3 -> 0.1
- rule via_min_size: 0.4 -> 0.45

Commit message: PCB layout work
Parts:
- moved R614 75.3 mm to (108.3, 36.5)
- moved C437 68.8 mm to (77.3, 70.7)
- moved C439 62.8 mm to (67.5, 80.3), turned to 90 degrees
- moved C438 61.3 mm to (87.2, 81.0), turned to 90 degrees
- moved R610 53.3 mm to (143.9, 151.8)
- moved U601 45.3 mm to (136.6, 150.3)
- moved C607 43.3 mm to (139.9, 145.3)
- moved C608 41.4 mm to (126.5, 147.9)
- moved R603 39.8 mm to (89.8, 90.2)
- moved R604 39.4 mm to (94.8, 93.7)
- moved C603 35.3 mm to (130.1, 142.8)
- moved L406 31.4 mm to (71.8, 96.9)
- moved R302 30.7 mm to (58.1, 80.1)
- moved C304 25.3 mm to (59.4, 86.8)
- moved R605 21.7 mm to (89.8, 85.8)
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Connections:
- net Net-(P601-Pad13) renamed /Ports/PA4_P
- net Net-(P601-Pad14) renamed /Ports/PA4_N
- net Net-(P601-Pad15) renamed /Ports/PA5_P
- net Net-(P601-Pad16) renamed /Ports/PA5_N
- net Net-(P603-Pad15) renamed /Ports/PC5_P
- net Net-(P603-Pad16) renamed /Ports/PC5_N
- net Net-(P604-Pad11) renamed /Ports/PD3_P
- net Net-(P604-Pad12) renamed /Ports/PD3_N
- net Net-(R604-Pad1) renamed /Ports/FPGA_B4_N
- net Net-(R604-Pad2) renamed /Ports/FPGA_B4_P
- net Net-(R604-Pad3) renamed /Ports/FPGA_B5_N
- net Net-(R604-Pad4) renamed /Ports/FPGA_B5_P
- net Net-(R609-Pad3) renamed /Ports/FPGA_B16_N
- net Net-(R609-Pad4) renamed /Ports/FPGA_B16_P
- net Net-(R612-Pad3) renamed /Ports/FPGA_B20_N
- net Net-(R612-Pad4) renamed /Ports/FPGA_B20_P
- P601 pad 10: Net-(P601-Pad10) -> /Ports/PA2_N
- P601 pad 11: Net-(P601-Pad11) -> /Ports/PA3_P
- P601 pad 12: Net-(P601-Pad12) -> /Ports/PA3_N
- P601 pad 7: Net-(P601-Pad7) -> /Ports/PA1_P
- P601 pad 8: Net-(P601-Pad8) -> /Ports/PA1_N
- P601 pad 9: Net-(P601-Pad9) -> /Ports/PA2_P
- P602 pad 10: Net-(P602-Pad10) -> /Ports/PB2_N
- P602 pad 11: Net-(P602-Pad11) -> /Ports/PB3_P
- P602 pad 12: Net-(P602-Pad12) -> /Ports/PB3_N
- P602 pad 13: Net-(P602-Pad13) -> /Ports/PB4_P
- P602 pad 14: Net-(P602-Pad14) -> /Ports/PB4_N
- P602 pad 15: Net-(P602-Pad15) -> /Ports/PB5_P
- P602 pad 16: Net-(P602-Pad16) -> /Ports/PB5_N
- P602 pad 7: Net-(P602-Pad7) -> /Ports/PB1_P
- P602 pad 8: Net-(P602-Pad8) -> /Ports/PB1_N
- P602 pad 9: Net-(P602-Pad9) -> /Ports/PB2_P
- P603 pad 10: Net-(P603-Pad10) -> /Ports/PC2_N
- P603 pad 11: Net-(P603-Pad11) -> /Ports/PC3_P
- P603 pad 12: Net-(P603-Pad12) -> /Ports/PC3_N
- P603 pad 13: Net-(P603-Pad13) -> /Ports/PC4_P
- P603 pad 14: Net-(P603-Pad14) -> /Ports/PC4_N
- P603 pad 7: Net-(P603-Pad7) -> /Ports/PC1_P
- P603 pad 8: Net-(P603-Pad8) -> /Ports/PC1_N
- P603 pad 9: Net-(P603-Pad9) -> /Ports/PC2_P
- P604 pad 10: Net-(P604-Pad10) -> /Ports/PD2_N
- P604 pad 13: Net-(P604-Pad13) -> /Ports/PD4_P
- P604 pad 14: Net-(P604-Pad14) -> /Ports/PD4_N
- P604 pad 15: Net-(P604-Pad15) -> /Ports/PD5_P
- P604 pad 16: Net-(P604-Pad16) -> /Ports/PD5_N
- P604 pad 7: Net-(P604-Pad7) -> /Ports/PD1_P
- P604 pad 8: Net-(P604-Pad8) -> /Ports/PD1_N
- P604 pad 9: Net-(P604-Pad9) -> /Ports/PD2_P
- R201 pad 1: /SDRAM/SDRAM_D0 -> /SDRAM/SDRAM_D1
- R201 pad 2: /SDRAM/SDRAM_D1 -> /SDRAM/SDRAM_D0
- R201 pad 3: /SDRAM/SDRAM_D2 -> /SDRAM/SDRAM_D3
- R201 pad 4: /SDRAM/SDRAM_D3 -> /SDRAM/SDRAM_D4
- R202 pad 1: /SDRAM/SDRAM_D4 -> /SDRAM/SDRAM_D7
- R202 pad 2: /SDRAM/SDRAM_D5 -> /SDRAM/SDRAM_D6
- R202 pad 3: /SDRAM/SDRAM_D6 -> /SDRAM/SDRAM_D5
- R202 pad 4: /SDRAM/SDRAM_D7 -> /SDRAM/SDRAM_D2
- R203 pad 5: /SDRAM/SDRAM_D8 -> /SDRAM/SDRAM_D13
- R203 pad 6: /SDRAM/SDRAM_D9 -> /SDRAM/SDRAM_D10
- R203 pad 7: /SDRAM/SDRAM_D10 -> /SDRAM/SDRAM_D9
- R203 pad 8: /SDRAM/SDRAM_D11 -> /SDRAM/SDRAM_D8
- R204 pad 5: /SDRAM/SDRAM_D12 -> /SDRAM/SDRAM_D11
- R204 pad 6: /SDRAM/SDRAM_D13 -> /SDRAM/SDRAM_D12
- R204 pad 7: /SDRAM/SDRAM_D14 -> /SDRAM/SDRAM_D15
- R204 pad 8: /SDRAM/SDRAM_D15 -> /SDRAM/SDRAM_D14
- R205 pad 1: /SDRAM/SDRAM_D16 -> /SDRAM/SDRAM_D17
- R205 pad 2: /SDRAM/SDRAM_D17 -> /SDRAM/SDRAM_D16
- R205 pad 3: /SDRAM/SDRAM_D18 -> /SDRAM/SDRAM_D19
- R205 pad 4: /SDRAM/SDRAM_D19 -> /SDRAM/SDRAM_D20
- R206 pad 1: /SDRAM/SDRAM_D20 -> /SDRAM/SDRAM_D23
- R206 pad 2: /SDRAM/SDRAM_D21 -> /SDRAM/SDRAM_D22
- R206 pad 3: /SDRAM/SDRAM_D22 -> /SDRAM/SDRAM_D21
- R206 pad 4: /SDRAM/SDRAM_D23 -> /SDRAM/SDRAM_D18
- R207 pad 5: /SDRAM/SDRAM_D24 -> /SDRAM/SDRAM_D29
- R207 pad 6: /SDRAM/SDRAM_D25 -> /SDRAM/SDRAM_D26
- R207 pad 7: /SDRAM/SDRAM_D26 -> /SDRAM/SDRAM_D25
- R207 pad 8: /SDRAM/SDRAM_D27 -> /SDRAM/SDRAM_D24
- R208 pad 5: /SDRAM/SDRAM_D28 -> /SDRAM/SDRAM_D27
- R208 pad 6: /SDRAM/SDRAM_D29 -> /SDRAM/SDRAM_D28
- R208 pad 7: /SDRAM/SDRAM_D30 -> /SDRAM/SDRAM_D31
- R208 pad 8: /SDRAM/SDRAM_D31 -> /SDRAM/SDRAM_D30
- R507 pad 3: Net-(C601-Pad1) -> (no net)
- R507 pad 4: GND -> (no net)
- R507 pad 5: Net-(C603-Pad1) -> (no net)
- R507 pad 6: Net-(C603-Pad1) -> (no net)
- R602 pad 1: Net-(C604-Pad1) -> /Ports/FPGA_B10_N
- R602 pad 2: Net-(R602-Pad2) -> /Ports/FPGA_B10_P
- R602 pad 3: Net-(R602-Pad3) -> /Ports/FPGA_B7_N
- R602 pad 4: Net-(R602-Pad4) -> /Ports/FPGA_B7_P
- R602 pad 5: Net-(P601-Pad7) -> /Ports/PB2_P
- R602 pad 6: Net-(P601-Pad8) -> /Ports/PB2_N
- R602 pad 7: Net-(P601-Pad2) -> /Ports/PB5_P
- R602 pad 8: Net-(R602-Pad8) -> /Ports/PB5_N
- R603 pad 1: Net-(R603-Pad1) -> /Ports/FPGA_B6_N
- R603 pad 2: Net-(R603-Pad2) -> /Ports/FPGA_B6_P
- R603 pad 3: Net-(R603-Pad3) -> /Ports/FPGA_B2_P
- R603 pad 4: Net-(R603-Pad4) -> /Ports/FPGA_B2_N
- R603 pad 5: Net-(P601-Pad11) -> /Ports/PA2_N
- R603 pad 6: Net-(P601-Pad12) -> /Ports/PA2_P
- R603 pad 7: Net-(P601-Pad9) -> /Ports/PB1_P
- R603 pad 8: Net-(P601-Pad10) -> /Ports/PB1_N
- R605 pad 1: Net-(R605-Pad1) -> Net-(C604-Pad1)
- R605 pad 3: Net-(R605-Pad3) -> /Ports/FPGA_B8_N
- R605 pad 4: Net-(R605-Pad4) -> /Ports/FPGA_B8_P
- R605 pad 5: Net-(P602-Pad9) -> /Ports/PB3_P
- R605 pad 6: Net-(P602-Pad10) -> /Ports/PB3_N
- R605 pad 7: Net-(P602-Pad7) -> Net-(P601-Pad2)
- R605 pad 8: Net-(P602-Pad8) -> Net-(R605-Pad8)
- R606 pad 1: Net-(R606-Pad1) -> /Ports/FPGA_B1_N
- R606 pad 2: Net-(R606-Pad2) -> /Ports/FPGA_B1_P
- R606 pad 3: Net-(R606-Pad3) -> /Ports/FPGA_B3_P
- R606 pad 4: Net-(R606-Pad4) -> /Ports/FPGA_B3_N
- R606 pad 5: Net-(P602-Pad13) -> /Ports/PA3_N
- R606 pad 6: Net-(P602-Pad14) -> /Ports/PA3_P
- R606 pad 7: Net-(P602-Pad11) -> /Ports/PA1_P
- R606 pad 8: Net-(P602-Pad12) -> /Ports/PA1_N
- R607 pad 1: Net-(R607-Pad1) -> /Ports/FPGA_B13_P
- R607 pad 2: Net-(R607-Pad2) -> /Ports/FPGA_B13_N
- R607 pad 3: Net-(R607-Pad3) -> /Ports/FPGA_B11_P
- R607 pad 4: Net-(R607-Pad4) -> /Ports/FPGA_B11_N
- R607 pad 5: Net-(P603-Pad7) -> /Ports/PC1_N
- R607 pad 6: Net-(P603-Pad8) -> /Ports/PC1_P
- R607 pad 7: Net-(P602-Pad15) -> /Ports/PC3_N
- R607 pad 8: Net-(P602-Pad16) -> /Ports/PC3_P
- R608 pad 1: Net-(R608-Pad1) -> /Ports/FPGA_B14_P
- R608 pad 2: Net-(R608-Pad2) -> /Ports/FPGA_B14_N
- R608 pad 3: Net-(R608-Pad3) -> /Ports/FPGA_B9_P
- R608 pad 4: Net-(R608-Pad4) -> /Ports/FPGA_B9_N
- R608 pad 5: Net-(P603-Pad11) -> /Ports/PB4_N
- R608 pad 6: Net-(P603-Pad12) -> /Ports/PB4_P
- R608 pad 7: Net-(P603-Pad9) -> /Ports/PC4_N
- R608 pad 8: Net-(P603-Pad10) -> /Ports/PC4_P
- R609 pad 1: Net-(R609-Pad1) -> /Ports/FPGA_B19_P
- R609 pad 2: Net-(R609-Pad2) -> /Ports/FPGA_B19_N
- R609 pad 7: Net-(P603-Pad13) -> /Ports/PD2_N
- R609 pad 8: Net-(P603-Pad14) -> /Ports/PD2_P
- R610 pad 3: (no net) -> Net-(C601-Pad1)
- R610 pad 4: (no net) -> GND
- R610 pad 5: (no net) -> Net-(C603-Pad1)
- R610 pad 6: (no net) -> Net-(C603-Pad1)
- R611 pad 1: Net-(C609-Pad1) -> /Ports/FPGA_B18_P
- R611 pad 2: Net-(R611-Pad2) -> /Ports/FPGA_B18_N
- R611 pad 3: Net-(R611-Pad3) -> /Ports/FPGA_B12_N
- R611 pad 4: Net-(R611-Pad4) -> /Ports/FPGA_B12_P
- R611 pad 5: Net-(P604-Pad7) -> /Ports/PC2_P
- R611 pad 6: Net-(P604-Pad8) -> /Ports/PC2_N
- R611 pad 7: Net-(P604-Pad2) -> /Ports/PD1_N
- R611 pad 8: Net-(R611-Pad8) -> /Ports/PD1_P
- R612 pad 1: Net-(R612-Pad1) -> /Ports/FPGA_B27_P
- R612 pad 2: Net-(R612-Pad2) -> /Ports/FPGA_B27_N
- R612 pad 7: Net-(P604-Pad9) -> /Ports/PD5_N
- R612 pad 8: Net-(P604-Pad10) -> /Ports/PD5_P
- R613 pad 1: Net-(R613-Pad1) -> Net-(C609-Pad1)
- R613 pad 2: Net-(R613-Pad2) -> /Ports/FPGA_B21_N
- R613 pad 3: Net-(R613-Pad3) -> /Ports/FPGA_B21_P
- R613 pad 5: Net-(P604-Pad15) -> Net-(P604-Pad2)
- R613 pad 6: Net-(P604-Pad16) -> /Ports/PD4_P
- R613 pad 7: Net-(P604-Pad13) -> /Ports/PD4_N
- R613 pad 8: Net-(P604-Pad14) -> Net-(R613-Pad8)
- U201 pad A13: /SDRAM/SDRAM_D31 -> /SDRAM/SDRAM_D27
- U201 pad A14: /SDRAM/SDRAM_D0 -> /SDRAM/SDRAM_D31
- U201 pad B13: /SDRAM/~SDRAM_RAS~ -> /SDRAM/SDRAM_D28
- U201 pad B16: /SDRAM/SDRAM_A1 -> /SDRAM/SDRAM_D29
- U201 pad C12: /SDRAM/SDRAM_D3 -> /SDRAM/SDRAM_DQM1
- U201 pad C13: /SDRAM/SDRAM_D4 -> /SDRAM/SDRAM_A9
- U201 pad C15: /SDRAM/SDRAM_A11 -> /SDRAM/SDRAM_D30
- U201 pad C16: /SDRAM/SDRAM_D15 -> /SDRAM/SDRAM_D26
- U201 pad D12: /SDRAM/SDRAM_D2 -> /SDRAM/SDRAM_BA0
- U201 pad D15: /SDRAM/SDRAM_A0 -> /SDRAM/SDRAM_D25
- U201 pad D16: /SDRAM/SDRAM_D20 -> /SDRAM/SDRAM_D24
- U201 pad E11: /SDRAM/SDRAM_D1 -> /SDRAM/SDRAM_A5
- U201 pad E14: /SDRAM/SDRAM_D29 -> /SDRAM/SDRAM_A1
- U201 pad E15: /SDRAM/SDRAM_CKE -> /SDRAM/SDRAM_D23
- U201 pad E16: /SDRAM/~SDRAM_CAS~ -> /SDRAM/SDRAM_D22
- U201 pad F11: /SDRAM/SDRAM_D6 -> /SDRAM/SDRAM_D20
- U201 pad F12: /SDRAM/SDRAM_D5 -> /SDRAM/SDRAM_D11
- U201 pad F14: /SDRAM/SDRAM_D30 -> /SDRAM/SDRAM_A11
- U201 pad F16: /SDRAM/SDRAM_D25 -> /SDRAM/SDRAM_D21
- U201 pad G11: /SDRAM/SDRAM_D28 -> /SDRAM/SDRAM_A8
- U201 pad G12: /SDRAM/SDRAM_D27 -> /SDRAM/~SDRAM_CAS~
- U201 pad G14: /SDRAM/SDRAM_D24 -> /SDRAM/SDRAM_A4
- U201 pad G15: /SDRAM/SDRAM_D23 -> /SDRAM/SDRAM_D18
- U201 pad G16: /SDRAM/SDRAM_D26 -> /SDRAM/SDRAM_D17
- U201 pad H11: /SDRAM/SDRAM_D22 -> /SDRAM/~SDRAM_RAS~
- U201 pad H12: /SDRAM/SDRAM_D21 -> /SDRAM/SDRAM_A0
- U201 pad H15: /SDRAM/SDRAM_D14 -> /SDRAM/SDRAM_D16
- U201 pad H16: /SDRAM/SDRAM_D13 -> /SDRAM/SDRAM_D19
- U201 pad J14: /SDRAM/SDRAM_D11 -> /SDRAM/SDRAM_D15
- U201 pad K11: /SDRAM/SDRAM_D18 -> /SDRAM/SDRAM_CKE
- U201 pad K15: /SDRAM/SDRAM_A4 -> /SDRAM/SDRAM_D14
- U201 pad L10: Net-(R613-Pad4) -> /Ports/FPGA_B27_P
- U201 pad L15: /SDRAM/SDRAM_D19 -> /SDRAM/SDRAM_D10
- U201 pad L16: /SDRAM/SDRAM_DQM1 -> /SDRAM/SDRAM_D13
- U201 pad L7: Net-(R603-Pad4) -> /Ports/FPGA_B3_P
- U201 pad L8: Net-(R606-Pad4) -> /Ports/FPGA_B9_P
- U201 pad M11: Net-(R613-Pad3) -> /Ports/FPGA_B27_N
- U201 pad M14: /SDRAM/SDRAM_D16 -> /SDRAM/~SDRAM_CS~
- U201 pad M15: /SDRAM/SDRAM_D17 -> /SDRAM/SDRAM_D8
- U201 pad M16: /SDRAM/~SDRAM_CS~ -> /SDRAM/SDRAM_D9
- U201 pad M6: Net-(R603-Pad3) -> /Ports/FPGA_B3_N
- U201 pad M7: Net-(R606-Pad3) -> /Ports/FPGA_B9_N
- U201 pad M8: Net-(R609-Pad1) -> /Ports/FPGA_B14_N
- U201 pad M9: Net-(R609-Pad2) -> /Ports/FPGA_B14_P
- U201 pad N14: /SDRAM/SDRAM_A9 -> /SDRAM/SDRAM_BA1
- U201 pad N16: /SDRAM/SDRAM_BA1 -> /SDRAM/SDRAM_D7
- U201 pad N5: Net-(R602-Pad4) -> /Ports/FPGA_B1_P
- U201 pad P10: Net-(R611-Pad3) -> /Ports/FPGA_B18_N
- U201 pad P11: Net-(R611-Pad4) -> /Ports/FPGA_B18_P
- U201 pad P12: Net-(R613-Pad2) -> /Ports/FPGA_B21_P
- U201 pad P13: Net-(R613-Pad1) -> /Ports/FPGA_B21_N
- U201 pad P14: /SDRAM/SDRAM_D8 -> /SDRAM/SDRAM_D0
- U201 pad P15: /SDRAM/SDRAM_A8 -> /SDRAM/SDRAM_D5
- U201 pad P16: /SDRAM/SDRAM_BA0 -> /SDRAM/SDRAM_D6
- U201 pad P2: Net-(R603-Pad1) -> /Ports/FPGA_B2_N
- U201 pad P4: Net-(R602-Pad3) -> /Ports/FPGA_B1_N
- U201 pad P6: Net-(R607-Pad2) -> /Ports/FPGA_B10_P
- U201 pad P8: Net-(R608-Pad2) -> /Ports/FPGA_B12_P
- U201 pad P9: Net-(R608-Pad1) -> /Ports/FPGA_B12_N
- U201 pad R1: Net-(R603-Pad2) -> /Ports/FPGA_B2_P
- U201 pad R11: Net-(R612-Pad1) -> /Ports/FPGA_B19_N
- U201 pad R12: Net-(R612-Pad2) -> /Ports/FPGA_B19_P
- U201 pad R14: /SDRAM/SDRAM_D9 -> /SDRAM/SDRAM_D4
- U201 pad R15: /SDRAM/SDRAM_D7 -> /SDRAM/SDRAM_D2
- U201 pad R5: Net-(R605-Pad4) -> /Ports/FPGA_B7_P
- U201 pad R6: Net-(R605-Pad3) -> /Ports/FPGA_B7_N
- U201 pad R7: Net-(R607-Pad1) -> /Ports/FPGA_B10_N
- U201 pad R8: Net-(R607-Pad4) -> /Ports/FPGA_B11_P
- U201 pad R9: Net-(R608-Pad4) -> /Ports/FPGA_B13_P
- U201 pad T12: Net-(R611-Pad2) -> Net-(R613-Pad4)
- U201 pad T14: /SDRAM/SDRAM_D10 -> /SDRAM/SDRAM_D3
- U201 pad T15: /SDRAM/SDRAM_A5 -> /SDRAM/SDRAM_D1
- U201 pad T2: Net-(R605-Pad2) -> /Ports/FPGA_B6_P
- U201 pad T3: Net-(R605-Pad1) -> /Ports/FPGA_B6_N
- U201 pad T4: Net-(R606-Pad2) -> /Ports/FPGA_B8_P
- U201 pad T5: Net-(R606-Pad1) -> /Ports/FPGA_B8_N
- U201 pad T6: Net-(R602-Pad2) -> Net-(R605-Pad2)
- U201 pad T8: Net-(R607-Pad3) -> /Ports/FPGA_B11_N
- U201 pad T9: Net-(R608-Pad3) -> /Ports/FPGA_B13_N
- U202 pad 10: Net-(R202-Pad7) -> Net-(R202-Pad6)
- U202 pad 11: Net-(R202-Pad6) -> Net-(R202-Pad7)
- U202 pad 13: Net-(R202-Pad5) -> Net-(R202-Pad8)
- U202 pad 2: Net-(R201-Pad8) -> Net-(R201-Pad7)
- U202 pad 4: Net-(R201-Pad7) -> Net-(R201-Pad8)
- U202 pad 42: Net-(R203-Pad4) -> Net-(R203-Pad1)
- U202 pad 44: Net-(R203-Pad3) -> Net-(R203-Pad2)
- U202 pad 45: Net-(R203-Pad2) -> Net-(R203-Pad3)
- U202 pad 47: Net-(R203-Pad1) -> Net-(R204-Pad4)
- U202 pad 48: Net-(R204-Pad4) -> Net-(R204-Pad3)
- U202 pad 5: Net-(R201-Pad6) -> Net-(R202-Pad5)
- U202 pad 50: Net-(R204-Pad3) -> Net-(R203-Pad4)
- U202 pad 51: Net-(R204-Pad2) -> Net-(R204-Pad1)
- U202 pad 53: Net-(R204-Pad1) -> Net-(R204-Pad2)
- U202 pad 7: Net-(R201-Pad5) -> Net-(R201-Pad6)
- U202 pad 8: Net-(R202-Pad8) -> Net-(R201-Pad5)
- U203 pad 10: Net-(R206-Pad7) -> Net-(R206-Pad6)
- U203 pad 11: Net-(R206-Pad6) -> Net-(R206-Pad7)
- U203 pad 13: Net-(R206-Pad5) -> Net-(R206-Pad8)
- U203 pad 2: Net-(R205-Pad8) -> Net-(R205-Pad7)
- U203 pad 4: Net-(R205-Pad7) -> Net-(R205-Pad8)
- U203 pad 42: Net-(R207-Pad4) -> Net-(R207-Pad1)
- U203 pad 44: Net-(R207-Pad3) -> Net-(R207-Pad2)
- U203 pad 45: Net-(R207-Pad2) -> Net-(R207-Pad3)
- U203 pad 47: Net-(R207-Pad1) -> Net-(R208-Pad4)
- U203 pad 48: Net-(R208-Pad4) -> Net-(R208-Pad3)
- U203 pad 5: Net-(R205-Pad6) -> Net-(R206-Pad5)
- U203 pad 50: Net-(R208-Pad3) -> Net-(R207-Pad4)
- U203 pad 51: Net-(R208-Pad2) -> Net-(R208-Pad1)
- U203 pad 53: Net-(R208-Pad1) -> Net-(R208-Pad2)
- U203 pad 7: Net-(R205-Pad5) -> Net-(R205-Pad6)
- U203 pad 8: Net-(R206-Pad8) -> Net-(R205-Pad5)
- U601 pad 1: Net-(R602-Pad8) -> Net-(R605-Pad8)
- U601 pad 2: Net-(R602-Pad8) -> Net-(R605-Pad8)
- U601 pad 6: Net-(R611-Pad8) -> Net-(R613-Pad8)
- U601 pad 7: Net-(R611-Pad8) -> Net-(R613-Pad8)
Routing:
- net GND: track 35.4 -> 107.5 mm, vias 0 -> 26
- net VCCIO_MCU: track 11.4 -> 49.8 mm, vias 0 -> 8
- net /Ports/FPGA_B3_P: track 0.00 -> 25.0 mm, vias 0 -> 2
- net /Ports/FPGA_B27_P: track 0.00 -> 24.1 mm, vias 0 -> 2
- net /Ports/FPGA_B3_N: track 0.00 -> 23.8 mm, vias 0 -> 2
- net /SDRAM/SDRAM_D4: track 0.00 -> 23.4 mm
- net +1V2: track 0.00 -> 22.5 mm, vias 0 -> 3
- net /Ports/FPGA_B27_N: track 0.00 -> 22.3 mm, vias 0 -> 2
- net /SDRAM/SDRAM_D0: track 0.00 -> 22.2 mm
- net /SDRAM/SDRAM_D28: track 0.00 -> 21.6 mm
- net /Ports/FPGA_B20_P: track 0.00 -> 21.5 mm, vias 0 -> 2
- net /Ports/FPGA_B1_P: track 0.00 -> 21.2 mm, vias 0 -> 2
- net /SDRAM/SDRAM_D27: track 0.00 -> 21.1 mm
- net /SDRAM/SDRAM_D3: track 0.00 -> 20.2 mm
- net /SDRAM/SDRAM_D31: track 0.00 -> 19.8 mm
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- added copper zone on In1.Cu, net GND
Other:
- net class Default: clearance 0.125 -> 0.2; trace_width 0.125 -> 0.3
- net class FPGA added: clearance 0.15, trace_width 0.15, via_dia 0.5, via_drill 0.2
- net class Impedance 100 Ohm added: clearance 0.15, trace_width 0.25, via_dia 0.6, via_drill 0.3
- net class Power added: clearance 0.15, trace_width 0.4, via_dia 0.5, via_drill 0.2
- net class Standard Signal removed
- rule trace_clearance: 0.125 -> 0.2

Commit message: Layout work
Parts:
- added R519: 22k, Resistors_SMD:R_0603, F.Cu at (34.2, 129.8)
- moved Q402 90.0 mm to (54.0, 47.0)
- moved JP502 88.2 mm to (42.8, 63.2)
- moved R412 88.2 mm to (27.9, 91.8)
- moved C431 87.0 mm to (27.9, 88.0), turned to 180 degrees
- moved C434 86.1 mm to (27.9, 86.5), turned to 180 degrees
- moved P502 86.0 mm to (52.9, 131.8), turned to 90 degrees
- moved P501 83.2 mm to (40.2, 131.8), turned to 90 degrees
- moved C435 82.6 mm to (51.9, 83.4), turned to 180 degrees
- moved R408 80.4 mm to (22.1, 84.3), turned to 90 degrees
- moved R413 77.0 mm to (52.0, 86.9)
- moved R415 76.5 mm to (52.0, 85.3)
- moved C432 76.4 mm to (51.9, 81.9), turned to 180 degrees
- moved R409 75.5 mm to (23.8, 84.3), turned to 270 degrees
- moved R414 75.2 mm to (27.9, 90.1)
- moved L404 74.6 mm to (32.0, 83.6), turned to 270 degrees
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Connections:
- R302 pad 4: MCU_PWRINT -> (no net)
- R302 pad 5: VCCIO_MCU -> (no net)
- R402 pad 3: Net-(R402-Pad3) -> (no net)
- R402 pad 4: Net-(R402-Pad4) -> MCU_PWRINT
- R402 pad 5: +2V5 -> VCCIO_MCU
- R402 pad 6: +2V5 -> (no net)
- R501 pad 5: VCCIO_MCU -> +2V5
- R501 pad 6: VCCIO_MCU -> +2V5
- R505 pad 3: VCCBU_MCU -> VCCIO_MCU
- R505 pad 6: Net-(C509-Pad1) -> Net-(R505-Pad6)
- R506 pad 2: Net-(R506-Pad2) -> GND
- R506 pad 7: VCCIO_MCU -> Net-(R506-Pad7)
- R507 pad 1: GND -> VCCBU_MCU
- R507 pad 2: /Misc/HSMCI_MCCDA -> (no net)
- R507 pad 3: (no net) -> Net-(R507-Pad3)
- R507 pad 4: (no net) -> Net-(R507-Pad4)
- R507 pad 5: (no net) -> VCCIO_MCU
- R507 pad 6: (no net) -> VCCIO_MCU
- R507 pad 7: Net-(C515-Pad1) -> (no net)
- R507 pad 8: Net-(R507-Pad8) -> Net-(C509-Pad1)
- U201 pad G6: Net-(R402-Pad3) -> Net-(R501-Pad3)
- U201 pad H2: Net-(R402-Pad4) -> Net-(R501-Pad4)
- U302 pad 11: Net-(R501-Pad4) -> Net-(R507-Pad4)
- U302 pad 138: Net-(R507-Pad8) -> Net-(R506-Pad7)
- U302 pad 7: Net-(R506-Pad2) -> Net-(R505-Pad6)
- U501 pad 13: Net-(R506-Pad2) -> Net-(R505-Pad6)
- U501 pad 2: Net-(R402-Pad4) -> Net-(R501-Pad4)
- U502 pad 2: Net-(R402-Pad4) -> Net-(R501-Pad4)
- W501 pad 1: Net-(R402-Pad4) -> Net-(R501-Pad4)
- X501 pad 1: Net-(R501-Pad4) -> Net-(R507-Pad4)
- X501 pad 5: Net-(R506-Pad2) -> Net-(R505-Pad6)
- X501 pad 9: Net-(R501-Pad3) -> Net-(R507-Pad3)
Routing:
- net /Power Supply/VCC_SYS: track 11.4 -> 44.6 mm
- net Net-(C515-Pad1): track 0.00 -> 27.1 mm
- net +1V8: track 0.00 -> 24.6 mm, vias 0 -> 2
- net Net-(D505-Pad2): track 0.00 -> 20.6 mm
- net Net-(C419-Pad1): track 0.00 -> 20.0 mm
- net VCCIO_MCU: track 49.8 -> 68.2 mm
- net /Power Supply/VREF_2V5: track 0.00 -> 18.3 mm
- net Net-(C424-Pad1): track 0.00 -> 18.1 mm, vias 0 -> 4
- net Net-(P504-Pad3): track 0.00 -> 17.9 mm
- net Net-(P504-Pad2): track 0.00 -> 15.6 mm
- net /Misc/HSMCI_MCDA1: track 0.00 -> 15.5 mm
- net /Misc/HSMCI_MCDA0: track 0.00 -> 14.1 mm
- net Net-(C511-Pad1): track 0.00 -> 13.9 mm
- net +1V2: track 22.5 -> 36.0 mm, vias 3 -> 5
- net /Misc/HSMCI_MCCDA: track 0.00 -> 11.0 mm
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- added copper zone on F.Cu, net +1V2
- added copper zone on F.Cu, net GND
- added copper zone on F.Cu, net Net-(C424-Pad1)
- added copper zone on F.Cu, net Net-(L405-Pad1)
Other:
- rule pad_to_mask_clearance: 0.1 -> 0

Commit message: Layout work
Parts:
- R519: value 22k -> 10k
- moved U601 95.3 mm to (112.6, 58.1), turned to 180 degrees
- moved C608 94.6 mm to (112.6, 54.4)
- moved C607 91.5 mm to (117.6, 56.6), turned to 270 degrees
- moved C603 84.0 mm to (117.6, 59.8), turned to 90 degrees
- moved R610 59.4 mm to (120.0, 58.1)
- moved R302 38.2 mm to (38.0, 108.1)
- moved C509 34.8 mm to (70.3, 95.8), turned to 90 degrees
- moved JP501 29.0 mm to (73.2, 131.8)
- moved W502 27.5 mm to (90.3, 104.2)
- moved W504 27.4 mm to (85.3, 104.2)
- moved W503 25.4 mm to (87.8, 104.2)
- moved W501 22.3 mm to (92.8, 104.2)
- moved C304 15.2 mm to (73.8, 91.5)
- moved R301 14.4 mm to (50.3, 90.8), turned to 270 degrees
- moved X501 12.7 mm to (85.9, 131.8)
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Connections:
- JP501 pad 3: Net-(JP501-Pad3) -> +2V5
- JP501 pad 5: +2V5 -> Net-(JP501-Pad5)
- P502 pad 11: /Misc/MCU_TXD1 -> Net-(P502-Pad11)
- P502 pad 12: /Misc/MCU_RXD1 -> /Misc/MCU_TWCK1
- P502 pad 3: Net-(P502-Pad3) -> /Misc/MCU_TXD0
- P502 pad 4: /Misc/MCU_TWCK1 -> /Misc/MCU_SCK0
- P502 pad 5: /Misc/MCU_SCK0 -> /Misc/MCU_TXD1
- P502 pad 6: /Misc/MCU_TWD1 -> /Misc/MCU_RXD0
- P502 pad 7: /Misc/MCU_TXD0 -> /Misc/MCU_CTS1
- P502 pad 8: /Misc/MCU_CTS1 -> /Misc/MCU_RXD1
- P502 pad 9: /Misc/MCU_RXD0 -> /Misc/MCU_TWD1
- R301 pad 1: VCCIO_MCU -> GND
- R301 pad 5: /InterConnect/FPGA_CRC_ERROR -> /InterConnect/~FPGA_CONFIG~
- R301 pad 6: /InterConnect/FPGA_CONF_DONE -> /InterConnect/~FPGA_STATUS~
- R301 pad 7: /InterConnect/~FPGA_STATUS~ -> /InterConnect/~FPGA_CLR~
- R301 pad 8: /InterConnect/~FPGA_CLR~ -> /InterConnect/FPGA_DEV_OE
- R302 pad 3: GND -> VCCIO_MCU
- R302 pad 6: /InterConnect/FPGA_CONFIG_SEL -> /InterConnect/FPGA_CONF_DONE
- R302 pad 7: /InterConnect/FPGA_DEV_OE -> /InterConnect/FPGA_CONFIG_SEL
- R302 pad 8: /InterConnect/~FPGA_CONFIG~ -> /InterConnect/FPGA_CRC_ERROR
- R501 pad 1: GND -> Net-(R501-Pad1)
- R501 pad 7: +2V5 -> GND
- R501 pad 8: Net-(R501-Pad8) -> +2V5
- R503 pad 1: Net-(JP501-Pad6) -> Net-(JP501-Pad5)
- R504 pad 1: Net-(JP501-Pad4) -> Net-(JP501-Pad1)
- R505 pad 1: Net-(R505-Pad1) -> Net-(JP501-Pad6)
- R505 pad 2: Net-(JP501-Pad2) -> Net-(R505-Pad2)
- R505 pad 3: VCCIO_MCU -> Net-(R505-Pad3)
- R505 pad 4: Net-(JP501-Pad3) -> VCCIO_MCU
- R505 pad 5: VCCIO_MCU -> Net-(R505-Pad5)
- R505 pad 6: Net-(R505-Pad6) -> VCCIO_MCU
- R505 pad 7: VCCIO_MCU -> GND
- R506 pad 3: GND -> VCCBU_MCU
- R506 pad 6: Net-(R506-Pad6) -> Net-(C509-Pad1)
- R507 pad 1: VCCBU_MCU -> VCCIO_MCU
- R507 pad 3: Net-(R507-Pad3) -> VCCIO_MCU
- R507 pad 4: Net-(R507-Pad4) -> VCCIO_MCU
- R507 pad 5: VCCIO_MCU -> Net-(R507-Pad5)
- R507 pad 6: VCCIO_MCU -> Net-(JP501-Pad4)
- R507 pad 8: Net-(C509-Pad1) -> Net-(R507-Pad8)
- R610 pad 1: Net-(C605-Pad1) -> Net-(C607-Pad1)
- R610 pad 3: Net-(C601-Pad1) -> GND
- R610 pad 4: GND -> Net-(C603-Pad1)
- R610 pad 5: Net-(C603-Pad1) -> Net-(C601-Pad1)
- R610 pad 8: Net-(C607-Pad1) -> Net-(C605-Pad1)
- U201 pad G1: Net-(R501-Pad2) -> Net-(R501-Pad3)
- U201 pad G6: Net-(R501-Pad3) -> Net-(R501-Pad4)
- U201 pad H2: Net-(R501-Pad4) -> Net-(R501-Pad1)
- U201 pad H3: Net-(R501-Pad8) -> Net-(R501-Pad2)
- U302 pad 107: /Misc/~SD_CD~ -> Net-(P502-Pad11)
- U302 pad 11: Net-(R507-Pad4) -> Net-(R507-Pad5)
- U302 pad 4: Net-(JP501-Pad3) -> Net-(JP501-Pad6)
- U302 pad 45: Net-(P502-Pad3) -> /Misc/VBUS_DETECT
- U302 pad 46: Net-(U302-Pad46) -> /Misc/~SD_CD~
- U302 pad 48: /Misc/VBUS_DETECT -> Net-(U302-Pad48)
- U302 pad 7: Net-(R505-Pad6) -> Net-(R505-Pad3)
- U302 pad 9: Net-(R506-Pad6) -> Net-(R505-Pad2)
- U501 pad 10: Net-(JP501-Pad1) -> Net-(JP501-Pad2)
- U501 pad 11: Net-(JP501-Pad3) -> Net-(JP501-Pad6)
- U501 pad 12: Net-(R506-Pad6) -> Net-(R505-Pad2)
- U501 pad 13: Net-(R505-Pad6) -> Net-(R505-Pad3)
- U501 pad 2: Net-(R501-Pad4) -> Net-(R501-Pad1)
- U501 pad 3: Net-(R501-Pad8) -> Net-(R501-Pad2)
- U501 pad 4: Net-(R501-Pad2) -> Net-(R501-Pad3)
- U501 pad 8: Net-(JP501-Pad4) -> Net-(JP501-Pad1)
- U502 pad 2: Net-(R501-Pad4) -> Net-(R501-Pad1)
- U502 pad 3: Net-(R501-Pad8) -> Net-(R501-Pad2)
- U502 pad 4: Net-(R501-Pad2) -> Net-(R501-Pad3)
- U502 pad 8: Net-(JP501-Pad6) -> Net-(JP501-Pad5)
- W501 pad 1: Net-(R501-Pad4) -> Net-(R501-Pad1)
- W502 pad 1: Net-(R501-Pad8) -> Net-(R501-Pad2)
- W503 pad 1: Net-(R501-Pad2) -> Net-(R501-Pad3)
- X501 pad 1: Net-(R507-Pad4) -> Net-(R507-Pad5)
- X501 pad 2: Net-(JP501-Pad2) -> Net-(JP501-Pad4)
- X501 pad 3: Net-(R506-Pad6) -> Net-(R505-Pad2)
- X501 pad 4: Net-(R505-Pad1) -> Net-(R507-Pad8)
- X501 pad 5: Net-(R505-Pad6) -> Net-(R505-Pad3)
- X501 pad 9: Net-(R507-Pad3) -> Net-(R505-Pad5)
Routing:
- net GND: track 102.6 -> 163.0 mm, vias 3 -> 22
- net Net-(JP501-Pad5): track 0.00 -> 42.6 mm, vias 0 -> 1
- net ~MCU_NPCS1~: track 0.00 -> 34.6 mm
- net Net-(C601-Pad1): track 3.89 -> 36.5 mm
- net /Misc/MCU_RTS1: track 0.00 -> 22.2 mm, vias 0 -> 1
- net Net-(C605-Pad1): track 3.45 -> 23.4 mm
- net Net-(JP501-Pad6): track 1.94 -> 21.1 mm
- net Net-(JP501-Pad2): track 0.00 -> 18.9 mm
- net Net-(JP501-Pad1): track 0.00 -> 18.2 mm, vias 0 -> 1
- net Net-(P502-Pad11): track 0.00 -> 17.7 mm
- net /Misc/MCU_TWD1: track 0.00 -> 17.3 mm
- net /Misc/MCU_CTS1: track 0.00 -> 16.7 mm
- net /Misc/MCU_TXD0: track 0.00 -> 16.2 mm
- net /Misc/MCU_TXD1: track 0.00 -> 15.7 mm
- net VCCIO_MCU: track 68.2 -> 83.1 mm, vias 8 -> 13
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- added copper zone on F.Cu, net +1V8
- added copper zone on F.Cu, net Net-(L404-Pad1)
Other:
- net class Default: clearance 0.2 -> 0.15
- rule trace_clearance: 0.2 -> 0.15
