File: board/data-logger.kicad_pcb (KiCad board)
At the start: 6 copper layers, 294 parts, among them P201 CONN_01X02, P202 USB_B_3, P301 CONN_02X10, P302 CONN_02X10, P303 CONN_02X10, P601 CONN_02X05, P602 CONN_02X05, Q201 IRLML6344TRPBF, Q202 Q_NPN_BEC, SW201 SW_Push, U201 LM5050-1, U202 CYUSB3012-BZXC, U203 R3111xxxB, U204 SP3010-04UTG, U205 NCP6324B, U206 NCP6332B, U207 NCP6332B, U208 MIC23050-4YML, U209 MIC23050-SYML, U210 AP2138N-1.8TRG1, U301 5CEFA2F23, U302 LMC6062, U303 FSA5157P6X, U304 FSA5157P6X, U305 LMC6062, U306 FSA5157P6X, U401 IS43TR16256LA, U402 DSC1103CI5-100.0000, U403 NCP51200, U501 25LC_EEPROM, U502 LSF0108, U503 CDCE913, X501 CONN_DEBUG_MCNET, Y501 19.200MHz

Commit message: Initial layout work
Parts:
- moved C228 121.1 mm to (251.1, 162.0)
- moved C623 121.1 mm to (259.0, 182.5)
- moved L201 121.1 mm to (279.5, 176.0)
- moved R320 121.1 mm to (263.0, 178.5)
- moved C203 121.1 mm to (280.6, 164.5)
- moved C232 121.1 mm to (255.5, 146.1)
- moved C237 121.1 mm to (251.8, 156.0)
- moved C242 121.1 mm to (269.7, 147.6)
- moved C304 121.1 mm to (268.5, 152.8)
- moved C307 121.1 mm to (253.3, 164.0)
- moved C310 121.1 mm to (274.4, 143.0)
- moved C508 121.1 mm to (262.5, 160.9)
- moved C511 121.1 mm to (271.6, 173.5)
- moved C514 121.1 mm to (262.5, 173.9)
- moved C604 121.1 mm to (249.2, 178.5)
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Connections:
- C411 pad 1: /Cyclone V DDR3 RAM/VTT_DDR3 -> GND
- R403 pad 1: /Cyclone V DDR3 RAM/FPGA_DDR3_ODT -> /Cyclone V DDR3 RAM/~FPGA_DDR3_CS~
- R403 pad 2: /Cyclone V DDR3 RAM/~FPGA_DDR3_WE~ -> /Cyclone V DDR3 RAM/~FPGA_DDR3_CAS~
- R403 pad 3: /Cyclone V DDR3 RAM/~FPGA_DDR3_CAS~ -> /Cyclone V DDR3 RAM/FPGA_DDR3_ODT
- R404 pad 1: /Cyclone V DDR3 RAM/FPGA_DDR3_A6 -> /Cyclone V DDR3 RAM/FPGA_DDR3_A14
- R404 pad 2: /Cyclone V DDR3 RAM/FPGA_DDR3_A8 -> /Cyclone V DDR3 RAM/FPGA_DDR3_A1
- R404 pad 3: /Cyclone V DDR3 RAM/FPGA_DDR3_A11 -> /Cyclone V DDR3 RAM/FPGA_DDR3_A12
- R404 pad 4: /Cyclone V DDR3 RAM/FPGA_DDR3_A14 -> /Cyclone V DDR3 RAM/FPGA_DDR3_A10
- R405 pad 1: /Cyclone V DDR3 RAM/FPGA_DDR3_A10 -> Net-(R405-Pad1)
- R405 pad 2: /Cyclone V DDR3 RAM/FPGA_DDR3_A15 -> /Cyclone V DDR3 RAM/FPGA_DDR3_BA1
- R405 pad 3: /Cyclone V DDR3 RAM/FPGA_DDR3_BA1 -> /Cyclone V DDR3 RAM/FPGA_DDR3_A8
- R405 pad 4: /Cyclone V DDR3 RAM/FPGA_DDR3_A4 -> /Cyclone V DDR3 RAM/FPGA_DDR3_A11
- R406 pad 1: (no net) -> /Cyclone V DDR3 RAM/FPGA_DDR3_CKE
- R406 pad 2: /Cyclone V DDR3 RAM/FPGA_DDR3_CK_P -> /Cyclone V DDR3 RAM/FPGA_DDR3_A15
- R406 pad 3: /Cyclone V DDR3 RAM/FPGA_DDR3_CK_N -> /Cyclone V DDR3 RAM/FPGA_DDR3_A4
- R406 pad 4: /Cyclone V DDR3 RAM/FPGA_DDR3_CKE -> /Cyclone V DDR3 RAM/FPGA_DDR3_A6
- R406 pad 6: Net-(C410-Pad2) -> /Cyclone V DDR3 RAM/VTT_DDR3
- R406 pad 7: Net-(C410-Pad2) -> /Cyclone V DDR3 RAM/VTT_DDR3
- R407 pad 1: (no net) -> Net-(R407-Pad1)
- R407 pad 4: (no net) -> Net-(R407-Pad4)
- R407 pad 5: /Cyclone V DDR3 RAM/VTT_DDR3 -> GND
- R407 pad 8: /Cyclone V DDR3 RAM/VTT_DDR3 -> GND
- R408 pad 1: /Cyclone V DDR3 RAM/FPGA_DDR3_A9 -> /Cyclone V DDR3 RAM/FPGA_DDR3_A2
- R408 pad 2: /Cyclone V DDR3 RAM/FPGA_DDR3_A13 -> /Cyclone V DDR3 RAM/FPGA_DDR3_A9
- R408 pad 3: /Cyclone V DDR3 RAM/FPGA_DDR3_A7 -> /Cyclone V DDR3 RAM/FPGA_DDR3_A13
- R408 pad 4: /Cyclone V DDR3 RAM/FPGA_DDR3_A5 -> /Cyclone V DDR3 RAM/FPGA_DDR3_BA2
- R409 pad 1: /Cyclone V DDR3 RAM/FPGA_DDR3_A3 -> /Cyclone V DDR3 RAM/FPGA_DDR3_A7
- R409 pad 2: /Cyclone V DDR3 RAM/FPGA_DDR3_BA2 -> /Cyclone V DDR3 RAM/FPGA_DDR3_A5
- R409 pad 3: /Cyclone V DDR3 RAM/FPGA_DDR3_BA0 -> /Cyclone V DDR3 RAM/FPGA_DDR3_A3
- R409 pad 4: /Cyclone V DDR3 RAM/~FPGA_DDR3_CS~ -> /Cyclone V DDR3 RAM/FPGA_DDR3_BA0
- R410 pad 1: /Cyclone V DDR3 RAM/FPGA_DDR3_A1 -> /Cyclone V DDR3 RAM/FPGA_DDR3_CK_N
- R410 pad 2: /Cyclone V DDR3 RAM/FPGA_DDR3_A12 -> /Cyclone V DDR3 RAM/FPGA_DDR3_CK_P
- R410 pad 3: /Cyclone V DDR3 RAM/FPGA_DDR3_A0 -> /Cyclone V DDR3 RAM/~FPGA_DDR3_WE~
- R410 pad 4: /Cyclone V DDR3 RAM/FPGA_DDR3_A2 -> /Cyclone V DDR3 RAM/FPGA_DDR3_A0
- R410 pad 7: /Cyclone V DDR3 RAM/VTT_DDR3 -> Net-(C410-Pad2)
- R410 pad 8: /Cyclone V DDR3 RAM/VTT_DDR3 -> Net-(C410-Pad2)
- U202 pad A11: (no net) -> Net-(U202-PadA11)
- U202 pad C6: (no net) -> Net-(U202-PadC6)
- U202 pad C7: (no net) -> Net-(U202-PadC7)
- U202 pad C9: (no net) -> Net-(U202-PadC9)
- U202 pad D6: (no net) -> Net-(U202-PadD6)
- U202 pad H6: (no net) -> Net-(U202-PadH6)
- U202 pad K5: (no net) -> Net-(U202-PadK5)
- U203 pad 4: (no net) -> Net-(U203-Pad4)
- U203 pad 5: (no net) -> Net-(U203-Pad5)
- U206 pad 6: (no net) -> /FX3 USB & Power Supply/PG_1V35
- U301 pad A12: (no net) -> Net-(U301-PadA12)
- U301 pad A14: (no net) -> Net-(U301-PadA14)
- U301 pad A15: (no net) -> Net-(U301-PadA15)
- U301 pad A17: (no net) -> Net-(U301-PadA17)
- U301 pad A18: (no net) -> Net-(U301-PadA18)
- U301 pad A19: (no net) -> Net-(U301-PadA19)
- U301 pad A20: (no net) -> Net-(U301-PadA20)
- U301 pad A22: (no net) -> Net-(U301-PadA22)
- U301 pad AA17: (no net) -> Net-(U301-PadAA17)
- U301 pad AA18: (no net) -> Net-(U301-PadAA18)
- U301 pad AA19: (no net) -> Net-(U301-PadAA19)
- U301 pad AA20: (no net) -> Net-(U301-PadAA20)
- U301 pad AA22: (no net) -> Net-(U301-PadAA22)
- U301 pad AA5: (no net) -> Net-(U301-PadAA5)
- U301 pad AB12: (no net) -> Net-(U301-PadAB12)
- U301 pad AB20: (no net) -> Net-(U301-PadAB20)
- U301 pad AB21: (no net) -> Net-(U301-PadAB21)
- U301 pad AB22: (no net) -> Net-(U301-PadAB22)
- U301 pad AB3: (no net) -> Net-(U301-PadAB3)
- U301 pad AB6: (no net) -> /Cyclone V FX3 FIFO/FPGA_FX3_D4
- U301 pad B13: (no net) -> Net-(U301-PadB13)
- U301 pad B16: (no net) -> Net-(U301-PadB16)
- U301 pad B17: (no net) -> Net-(U301-PadB17)
- U301 pad B18: (no net) -> Net-(U301-PadB18)
- U301 pad B20: (no net) -> Net-(U301-PadB20)
- U301 pad B21: (no net) -> Net-(U301-PadB21)
- U301 pad B22: (no net) -> Net-(U301-PadB22)
- U301 pad B3: (no net) -> Net-(U301-PadB3)
- U301 pad B4: (no net) -> Net-(U301-PadB4)
- U301 pad B5: (no net) -> Net-(U301-PadB5)
- U301 pad C16: (no net) -> Net-(U301-PadC16)
- U301 pad C18: (no net) -> Net-(U301-PadC18)
- U301 pad C19: (no net) -> Net-(U301-PadC19)
- U301 pad C20: (no net) -> Net-(U301-PadC20)
- U301 pad C21: (no net) -> Net-(U301-PadC21)
- U301 pad D17: (no net) -> Net-(U301-PadD17)
- U301 pad D19: (no net) -> Net-(U301-PadD19)
- U301 pad D21: (no net) -> Net-(U301-PadD21)
- U301 pad D22: (no net) -> Net-(U301-PadD22)
- U301 pad D3: /Cyclone V Power/EXT_IO5 -> /Cyclone V Power/EXT_IO3
- U301 pad D9: (no net) -> Net-(U301-PadD9)
- U301 pad E10: (no net) -> Net-(U301-PadE10)
- U301 pad E15: (no net) -> Net-(U301-PadE15)
- U301 pad E16: (no net) -> Net-(U301-PadE16)
- U301 pad E17: (no net) -> Net-(U301-PadE17)
- U301 pad E19: (no net) -> Net-(U301-PadE19)
- U301 pad E2: /Cyclone V Power/EXT_IO4 -> /Cyclone V Power/EXT_IO2
- U301 pad E20: (no net) -> Net-(U301-PadE20)
- U301 pad E21: (no net) -> Net-(U301-PadE21)
- U301 pad E22: (no net) -> Net-(U301-PadE22)
- U301 pad E7: (no net) -> Net-(U301-PadE7)
- U301 pad F10: (no net) -> Net-(U301-PadF10)
- U301 pad F15: (no net) -> Net-(U301-PadF15)
- U301 pad F18: (no net) -> Net-(U301-PadF18)
- U301 pad F19: (no net) -> Net-(U301-PadF19)
- U301 pad F20: (no net) -> Net-(U301-PadF20)
- U301 pad F22: (no net) -> Net-(U301-PadF22)
- U301 pad F9: (no net) -> Net-(U301-PadF9)
- U301 pad G1: /Cyclone V Power/EXT_IO2 -> /Cyclone V Power/EXT_IO4
- U301 pad G10: (no net) -> Net-(U301-PadG10)
- U301 pad G17: (no net) -> Net-(U301-PadG17)
- U301 pad G18: (no net) -> Net-(U301-PadG18)
- U301 pad G2: /Cyclone V Power/EXT_IO3 -> /Cyclone V Power/EXT_IO5
- U301 pad G20: (no net) -> Net-(U301-PadG20)
- U301 pad G21: (no net) -> Net-(U301-PadG21)
- U301 pad G22: (no net) -> Net-(U301-PadG22)
- U301 pad H10: (no net) -> Net-(U301-PadH10)
- U301 pad H15: (no net) -> Net-(U301-PadH15)
- U301 pad H16: (no net) -> Net-(U301-PadH16)
- U301 pad H18: (no net) -> Net-(U301-PadH18)
- U301 pad H20: (no net) -> Net-(U301-PadH20)
- U301 pad H21: (no net) -> Net-(U301-PadH21)
- U301 pad J18: (no net) -> Net-(U301-PadJ18)
- U301 pad J21: (no net) -> Net-(U301-PadJ21)
- U301 pad J22: (no net) -> Net-(U301-PadJ22)
- U301 pad K19: (no net) -> Net-(U301-PadK19)
- U301 pad K20: (no net) -> Net-(U301-PadK20)
- U301 pad L9: (no net) -> Net-(U301-PadL9)
- U301 pad P14: (no net) -> Net-(U301-PadP14)
- U301 pad R14: (no net) -> Net-(U301-PadR14)
- U301 pad R4: (no net) -> Net-(U301-PadR4)
- U301 pad T14: (no net) -> Net-(U301-PadT14)
- U301 pad T4: (no net) -> Net-(U301-PadT4)
- U301 pad U15: (no net) -> Net-(U301-PadU15)
- U301 pad U16: (no net) -> Net-(U301-PadU16)
- U301 pad U17: (no net) -> Net-(U301-PadU17)
- U301 pad U20: (no net) -> Net-(U301-PadU20)
- U301 pad U21: (no net) -> Net-(U301-PadU21)
- U301 pad U22: (no net) -> Net-(U301-PadU22)
- U301 pad V11: (no net) -> Net-(U301-PadV11)
- U301 pad V18: (no net) -> Net-(U301-PadV18)
- U301 pad V19: (no net) -> Net-(U301-PadV19)
- U301 pad V20: (no net) -> Net-(U301-PadV20)
- U301 pad V21: (no net) -> Net-(U301-PadV21)
- U301 pad W19: (no net) -> Net-(U301-PadW19)
- U301 pad W21: (no net) -> Net-(U301-PadW21)
- U301 pad W22: (no net) -> Net-(U301-PadW22)
- U301 pad Y16: (no net) -> Net-(U301-PadY16)
- U301 pad Y17: (no net) -> Net-(U301-PadY17)
- U301 pad Y19: (no net) -> Net-(U301-PadY19)
- U301 pad Y20: (no net) -> Net-(U301-PadY20)
- U301 pad Y21: (no net) -> Net-(U301-PadY21)
- U301 pad Y22: (no net) -> Net-(U301-PadY22)
- U301 pad Y6: (no net) -> Net-(U301-PadY6)
- U401 pad J1: (no net) -> Net-(U401-PadJ1)
- U401 pad J9: (no net) -> Net-(U401-PadJ9)
- U401 pad L1: (no net) -> Net-(U401-PadL1)
- U401 pad L9: (no net) -> Net-(U401-PadL9)
- U402 pad 2: (no net) -> Net-(U402-Pad2)
- U503 pad 4: (no net) -> Net-(U503-Pad4)
- X501 pad 7: (no net) -> Net-(X501-Pad7)
Routing:
- net GND: track 18.3 -> 143.0 mm, vias 34 -> 129
- net VCC_1V35: track 1.87 -> 78.2 mm, vias 4 -> 59
- net /Cyclone V DDR3 RAM/VREF_DDR3: track 0.57 -> 53.8 mm, vias 1 -> 4
- net /Cyclone V DDR3 RAM/FPGA_DDR3_CKE: track 2.77 -> 34.3 mm, vias 1 -> 3
- net /Cyclone V DDR3 RAM/VTT_DDR3: track 0.00 -> 27.8 mm
- net /Cyclone V DDR3 RAM/FPGA_DDR3_D15: track 0.57 -> 27.8 mm, vias 1 -> 2
- net /Cyclone V DDR3 RAM/FPGA_DDR3_CK_P: track 4.62 -> 30.9 mm, vias 1 -> 2
- net /Cyclone V DDR3 RAM/FPGA_DDR3_CK_N: track 4.54 -> 30.0 mm, vias 1 -> 2
- net /Cyclone V DDR3 RAM/FPGA_DDR3_DM1: track 0.57 -> 25.2 mm, vias 1 -> 2
- net /Cyclone V Power/EXT_IO2: track 0.00 -> 22.7 mm, vias 0 -> 1
- net /Cyclone V Power/EXT_IO12: track 0.00 -> 21.9 mm, vias 0 -> 1
- net /Cyclone V Power/EXT_IO6: track 0.00 -> 21.9 mm, vias 0 -> 1
- net /Cyclone V DDR3 RAM/FPGA_DDR3_D3: track 0.57 -> 22.4 mm, vias 1 -> 2
- net /Cyclone V Power/EXT_IO0: track 0.00 -> 21.7 mm, vias 0 -> 1
- net /Cyclone V DDR3 RAM/FPGA_CLK10_P: track 0.00 -> 21.5 mm, vias 0 -> 2
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- added copper zone on F.Cu, net /Cyclone V DDR3 RAM/VTT_DDR3
- added copper zone on F.Cu, net /FX3 USB & Power Supply/VCC_IN
- added copper zone on F.Cu, net GND
- added copper zone on In4.Cu, net GND
- added copper zone on F.Cu, net Net-(L207-Pad1)
- added copper zone on B.Cu, net VCC_1V35
- added copper zone on F.Cu, net VCC_1V35
- added copper zone on In1.Cu, net VCC_2V50
- removed copper zone on B.Cu, net GND
- removed copper zone on In1.Cu, net VCC_1V35
Other:
- board outline added: 60 x 80 mm
- net class 50Ohm_Impedance added: clearance 0.102, trace_width 0.25, via_dia 0.46, via_drill 0.254

Commit message: Rework power supply and simplify some things
Parts:
- removed C221, C235, C238: 10µF, Capacitors_SMD:C_0603
- removed C230: 15pF, Capacitors_SMD:C_0402
- removed L206: 1µH, AMesser_Inductors:Bourns_SRN4018TA
- removed R211: 100k, Resistors_SMD:R_0603
- removed R212: 220k 1%, Resistors_SMD:R_0603
- removed R213: 261k 1%, Resistors_SMD:R_0603
- removed U205: NCP6324B, AMesser_Power_Management:ON_Semiconductor_WDFN-8_2x2mm_Pitch0.5mm
- added C243: 10µF/35V, Capacitors_SMD:C_1206, F.Cu at (69.0, 106.2)
- added C244: 22µF/4V, Capacitors_SMD:C_0603, F.Cu at (75.4, 109.6)
- added C245: 22µF/4V, Capacitors_SMD:C_0603, F.Cu at (75.4, 108.2)
- added C246: 220µF/6.3V, Capacitors_ThroughHole:CP_Radial_D5.0mm_P2.00mm, F.Cu at (75.0, 113.1)
- added L1: 4.7µH/2.8A, AMesser_Inductors:Bourns_SRN6045TA, F.Cu at (73.6, 104.3)
- added Q203: CSD17313Q2, AMesser_Transistors:Texas_Instruments_WSON-6_2x2mm-Q2, F.Cu at (69.0, 102.8)
- added Q204: CSD17313Q2, AMesser_Transistors:Texas_Instruments_WSON-6_2x2mm-Q2, F.Cu at (72.8, 108.9)
- added R218: 4.64k, Resistors_SMD:R_0603, F.Cu at (75.2, 116.8)
- added R219: 11k, Resistors_SMD:R_0603, F.Cu at (72.7, 116.8)
- added R220: 11k, Resistors_SMD:R_0603, F.Cu at (70.3, 111.5)
- added U211: TPS53015, Housings_SSOP:MSOP-10_3x3mm_Pitch0.5mm, F.Cu at (67.7, 113.3)
- C201: value 4.7µF -> 4.3µF/2.5V
- C240: value 10µF -> 1µF/35V
- C241: value 10µF -> 4.7µF/16V
- C242: value 10µF -> 0.1µF/16V; footprint Capacitors_SMD:C_0603 -> Capacitors_SMD:C_0402
- C613, C614, C615, C616, C618, C620, C624, C628: value 4µ7 -> 100nF
- moved C242 205.9 mm to (67.2, 109.8), turned to 180 degrees
- moved C601 194.9 mm to (99.3, 106.5), turned to 90 degrees
- moved C628 188.4 mm to (99.3, 116.7), turned to 90 degrees
- moved C602 176.4 mm to (99.3, 110.5), turned to 90 degrees
- moved C624 172.7 mm to (99.3, 118.8), turned to 270 degrees
- moved C603 165.1 mm to (96.8, 116.7), turned to 90 degrees
- moved C604 163.7 mm to (96.8, 118.8), turned to 270 degrees
- moved C217 100.9 mm to (123.5, 180.6)
- moved L204 66.0 mm to (56.8, 129.7)
- moved C620 61.2 mm to (99.3, 112.6), turned to 90 degrees
- moved C618 59.0 mm to (99.3, 114.7), turned to 270 degrees
- moved C240 58.3 mm to (70.3, 114.2), turned to 90 degrees
- moved C616 57.7 mm to (96.8, 112.6), turned to 90 degrees
- moved C607 55.7 mm to (98.5, 112.6), turned to 90 degrees
- moved C606 55.5 mm to (96.8, 114.7), turned to 270 degrees
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Connections:
- C240 pad 1: VCC_1V10 -> /FX3 USB & Power Supply/VCC_IN
- C241 pad 1: VCC_1V10 -> Net-(C241-Pad1)
- C242 pad 1: VCC_1V10 -> Net-(C242-Pad1)
- C242 pad 2: GND -> Net-(C242-Pad2)
Routing:
- net VCC_1V10: track 1.98 -> 24.9 mm, vias 4 -> 22
- net GND: track 143.0 -> 158.7 mm, vias 129 -> 140
- net VCC_3V30: track 0.93 -> 6.90 mm, vias 2 -> 6
- net /FX3 USB & Power Supply/VCC_IN: track 3.94 -> 9.76 mm
- net /Cyclone V Power/EXT_IO9: track 18.9 -> 19.6 mm
- net /FX3 USB & Power Supply/PG_1V35: track 0.64 -> 0.00 mm, vias 1 -> 0
- net (no net): vias 0 -> 1
- added copper zone on F.Cu, net VCC_1V10
